Commit message: Add workspace fetching

File: toy_gym/envs/urdf/maze_world_with_obs.urdf (robot description, URDF)
Before this commit: robot maze_world, 6 links, 5 joints
Links:
- added link obstacle2, mass 10; collision box size=0.5 0.5 1; visual box size=0.5 0.5 1
- link wall3: geometry collision box size=10 0.1 1; visual box size=10 0.1 1
- link wall4: geometry collision box size=10 0.1 1; visual box size=10 0.1 1
Joints:
- added joint base_to_obstacle2: type fixed, parent base_link, child obstacle2, origin xyz=0.0 4 0.0 rpy=0.0 0.0 0.0
- joint base_to_obstacle: origin xyz=-2.5 0.0 0.0 rpy=0.0 0.0 1.57075 -> xyz=-2.5 0.0 0.0 rpy=0.0 0.0 0.0
- joint base_to_wall3: origin xyz=0.0 -5.0 0.0 rpy=0.0 0.0 1.57075 -> xyz=0.0 -5.0 0.0 rpy=0.0 0.0 0
- joint base_to_wall4: origin xyz=0.0 5.0 0.0 rpy=0.0 0.0 1.57075 -> xyz=0.0 5.0 0.0 rpy=0.0 0.0 0
