Commit message: update urdf

File: toy_gym/envs/urdf/maze_world_narrow.urdf (robot description, URDF)
Before this commit: robot maze_world, 8 links, 7 joints
Links:
- link obstacle2: geometry collision box size=0.6 4 1; visual box size=0.6 4 1
- link obstacle3: geometry collision box size=2 0.6 1; visual box size=2 0.6 1
Joints:
- joint base_to_obstacle2: origin xyz=0.0 -4 0.0 rpy=0.0 0.0 0.0 -> xyz=0 -3 0.0 rpy=0.0 0.0 0.0
- joint base_to_obstacle3: origin xyz=3 0.0 0.0 rpy=0.0 0.0 0.0 -> xyz=4 -1 0.0 rpy=0.0 0.0 0.0
